Commit message: 修改了urdf 使得转向自如

File: src/robot_mrobot/mrobot_description/urdf/urobot.urdf (robot description, URDF)
Before this commit: robot urobot, 11 links, 10 joints
Joints:
- joint behindbase_to_frontbase: limit lower=-0.698 upper=0.698 effort=10000 velocity=0.1396 -> lower=-0.698 upper=0.698 effort=10000000 velocity=0.1396

Commit message: 把mpc算法中的模型换成了铰接车的

File: src/robot_mrobot/mrobot_description/urdf/urobot.urdf (robot description, URDF)
Before this commit: robot urobot, 11 links, 10 joints
Links:
- removed link gps_Link
Joints:
- removed joint gps_to_base

Commit message: 改成了四轮独驱动的模式 这样rviz中才能正常显示

File: src/robot_mrobot/mrobot_description/urdf/urobot.urdf (robot description, URDF)
Before this commit: robot urobot, 10 links, 9 joints
Joints:
- joint laser360_to_base: origin xyz=-0.728241888910018 0 0.533000000000001 rpy=0 0 0 -> xyz=-1.7 0 2.410 rpy=0 0 0; parent base_link -> behindbase_Link

Commit message: 改成了四轮独驱动的模式 这样rviz中才能正常显示

File: src/robot_mrobot/mrobot_description/urdf/urobot.urdf (robot description, URDF)
Before this commit: robot urobot, 10 links, 9 joints
Joints:
- joint laser360_to_base: origin xyz=-1.7 0 2.410 rpy=0 0 0 -> xyz=-0.4 0 1.2 rpy=0 0 0
